Commit message: [UPDATE 20241216]: add keypoint detection

File: CourseProject/PDM_urdf/Cross_cube_bottle.urdf (robot description, URDF)
Before this commit: robot Arrow_cube_cap, 1 links, 0 joints
Links:
- link baseLink: mass None -> .5; geometry collision mesh filename=Cross_cube_bottle2.obj scale=0.6 0.6 0.6; visual mesh filename=Cross_cube_bottle.obj scale=0.6 0.6 0.6

File: CourseProject/PDM_urdf/Cross_cube_cap.urdf (robot description, URDF)
Before this commit: robot Arrow_cube_cap, 1 links, 0 joints
Links:
- link baseLink: geometry collision mesh filename=Cross_cube_cap.obj scale=0.6 0.6 0.6; visual mesh filename=Cross_cube_cap.obj scale=0.6 0.6 0.6

File: CourseProject/PDM_urdf/Star_cube_bottle.urdf (robot description, URDF)
Before this commit: robot Arrow_cube_cap, 1 links, 0 joints
Links:
- link baseLink: mass None -> .5; geometry collision mesh filename=Star_cube_bottle.obj scale=0.6 0.6 0.6; visual mesh filename=Star_cube_bottle.obj scale=0.6 0.6 0.6

File: CourseProject/PDM_urdf/Star_cube_cap.urdf (robot description, URDF)
Before this commit: robot Arrow_cube_cap, 1 links, 0 joints
Links:
- link baseLink: geometry collision mesh filename=Star_cube_cap.obj scale=0.6 0.6 0.6; visual mesh filename=Star_cube_cap.obj scale=0.6 0.6 0.6
